File: hardware/power-manager.brd (EAGLE design)
At the start: 74 x 34 mm, 77 parts, among them IC1 ATMEGA168-AU, K1 G6J-2FL-Y, K2 G6J-2FL-Y, K3 G6J-2FL-Y, Q1 BSS138, Q2 BSS138, Q3 BSS138, U1 V_REG_LDOSMD, U2 INA219, U3 TPS2552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

Commit message: hw: rc2
Parts:
- added C20, C21, C22, C23: .1u, rcl:C0805
- added LED7: (no value), led:SML0805
- added R24, R25, R26, R27, R28, R29: 10k, rcl:R0603
- added R30: 330, rcl:R0603
- added R31: 100k, rcl:R0603
- U1: value V_REG_LDOSMD -> MIC5301
- moved R20 5.55 mm to (62.8, 30.9), flipped to the bottom, turned to 0 degrees
- moved C1 2.24 mm to (59.1, 8.53)
- moved C2 2.24 mm to (54.3, 8.53)
- moved JP1 2.03 mm to (52.4, 2.24)
- moved U1 1.83 mm to (56.7, 8.94)
- moved LED3 1.18 mm to (58.3, 30.9), turned to 0 degrees
- moved C6 1.09 mm to (63.0, 30.9), turned to 90 degrees
- moved C5 0.41 mm to (64.8, 30.9)
Connections:
- removed net LED_SYS: IC1.23, R20.1
- removed net N$21: K1.3, K1.6, X2.1
- new net POWER_ADC: C22.1, IC1.23, R28.2, R29.1
- new net POWER_IN: K1.3, K1.6, R28.1, X2.1
- new net USB1_ADC: C20.1, IC1.22, R24.2, R25.1
- new net USB1_IN: C9.1, JP1.1, R24.1, U$2.VBUS, U3.1
- new net USB2_ADC: C21.1, IC1.19, R26.2, R27.1
- new net USB2_IN: C11.1, R26.1, U$3.VBUS, U7.1
- net GND: now also C20.2, C21.2, C22.2, C23.2, LED7.C, R25.2, R27.2, R29.2, R31.2
- net MISO: now also R20.1
- net N$10: now also LED7.A, R30.2; no longer C11.1, U$3.VBUS, U7.1
- net N$19: now also R31.1
- net N$5: now also C23.1, U1.4; no longer C9.1, JP1.1, U$2.VBUS, U3.1
- net SCK: now also R30.1
Routing:
- net POWER_ADC: track 0.00 -> 60.1 mm, vias 0 -> 1
- net USB1_ADC: track 0.00 -> 51.7 mm, vias 0 -> 1
- net USB2_ADC: track 0.00 -> 50.1 mm, vias 0 -> 1
- net POWER_IN: track 0.00 -> 27.1 mm, vias 0 -> 1
- net USB1_IN: track 0.00 -> 26.7 mm, vias 0 -> 1
- net N$5: track 25.5 -> 1.75 mm
- net USB2_IN: track 0.00 -> 15.8 mm, vias 0 -> 1
- net N$21: track 9.44 -> 0.00 mm
- net N$10: track 10.4 -> 2.57 mm, vias 0 -> 1
- net MISO: track 3.91 -> 11.3 mm, vias 0 -> 1
- net SCK: track 11.1 -> 17.2 mm, vias 0 -> 1
- net LED_SYS: track 4.35 -> 0.00 mm
- net +5V: track 114.0 -> 110.5 mm
- net N$2: track 3.66 -> 2.28 mm
- net N$30: track 1.51 -> 2.57 mm, vias 0 -> 1
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Other:
- board text removed: "www.fabiobaltieri.com"

Commit message: hw: rc3
Parts:
- moved R10 0.20 mm to (48.2, 17.9)
- moved R14 0.20 mm to (31.5, 17.9)
- moved C10 0.20 mm to (45.9, 17.1)
- moved C12 0.20 mm to (29.3, 17.1)
- moved C14 0.20 mm to (51.4, 19.5)
- moved C15 0.20 mm to (34.7, 19.5)
- moved R11 0.20 mm to (50.4, 17.1)
- moved R13 0.20 mm to (31.5, 16.3)
- moved R15 0.20 mm to (33.7, 17.1)
- moved R9 0.20 mm to (48.2, 16.3)
Connections:
- net POWER_ADC: now also IC1.19; no longer IC1.23
- net USB1_ADC: now also IC1.23; no longer IC1.22
- net USB2_ADC: now also IC1.22; no longer IC1.19
Routing:
- net POWER_ADC: track 60.1 -> 57.0 mm
- net USB2_ADC: track 50.1 -> 52.4 mm
- net USB1_ADC: track 51.7 -> 52.7 mm

Commit message: hw: rc4?
Parts:
- moved JP2 2.76 mm to (3.05, 25.4), turned to 0 degrees
- moved JP3 1.92 mm to (10.6, 25.4), turned to 0 degrees
Routing:
- net N$26: track 12.8 -> 7.59 mm
- net N$23: track 8.91 -> 4.26 mm
- net IO1_EN: track 65.8 -> 69.3 mm
- net N$24: track 8.41 -> 10.1 mm
- net N$27: track 12.6 -> 13.5 mm
Changed lines of the file:
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@@
 <attribute name="VALUE" value="BSS138" x="-8.9408" y="-154.0764" size="1.778" layer="28" rot="MR0" display="off"/>
 </element>
-<element name="JP2" library="SparkFun-Connectors" package="1X02" value="" x="5.2832" y="27.0256" rot="R180"/>
+<element name="JP2" library="SparkFun-Connectors" package="1X02" value="" x="3.048" y="25.4"/>
 <element name="D3" library="diode" package="SOT23" value="BAT54" x="14.0208" y="19.9136" rot="MR180"/>
 <element name="K3" library="relay" package="G6J-2FL-Y" value="G6J-2FL-Y" x="16.6624" y="19.9136">
@@
 <attribute name="VALUE" value="BSS138" x="-1.778" y="-154.0764" size="1.778" layer="28" rot="MR0" display="off"/>
 </element>
-<element name="JP3" library="SparkFun-Connectors" package="1X02" value="" x="11.5824" y="27.0256" rot="R180"/>
+<element name="JP3" library="SparkFun-Connectors" package="1X02" value="" x="10.5664" y="25.4"/>
 <element name="R19" library="rcl" package="R0603" value="330" x="16.256" y="3.2512" rot="MR180"/>
 <element name="R20" library="rcl" package="R0603" value="330" x="62.7888" y="30.8864" rot="MR0"/>
@@
 <contactref element="Q2" pad="1"/>
 <wire x1="7.2492" y1="18.9136" x2="7.2492" y2="19.0348" width="0.2032" layer="16"/>
-<wire x1="7.2492" y1="19.0348" x2="16.0528" y2="27.8384" width="0.2032" layer="16"/>
-<wire x1="16.0528" y1="27.8384" x2="18.6944" y2="27.8384" width="0.2032" layer="16"/>
 <wire x1="18.6944" y1="27.8384" x2="19.5072" y2="28.6512" width="0.2032" layer="16"/>
 <wire x1="19.5072" y1="28.6512" x2="53.6448" y2="28.6512" width="0.2032" layer="16"/>
@@
 <wire x1="53.6448" y1="28.6512" x2="58.1152" y2="24.1808" width="0.2032" layer="16"/>
 <wire x1="58.1152" y1="24.1808" x2="64.4144" y2="24.1808" width="0.2032" layer="16"/>
+<wire x1="18.6944" y1="27.8384" x2="10.16" y2="27.8384" width="0.2032" layer="16"/>
+<wire x1="10.16" y1="27.8384" x2="8.3312" y2="26.0096" width="0.2032" layer="16"/>
+<wire x1="8.3312" y1="26.0096" x2="8.3312" y2="19.9956" width="0.2032" layer="16"/>
+<wire x1="8.3312" y1="19.9956" x2="7.2492" y2="18.9136" width="0.2032" layer="16"/>
 </signal>
 <signal name="N$23">
 <contactref element="JP2" pad="2"/>
 <contactref element="K2" pad="6"/>
-<wire x1="7.8896" y1="22.5136" x2="7.8896" y2="24.4192" width="0.4064" layer="1"/>
-<wire x1="7.8896" y1="24.4192" x2="7.5184" y2="24.7904" width="0.4064" layer="1"/>
-<wire x1="7.5184" y1="24.7904" x2="3.6576" y2="24.7904" width="0.4064" layer="1"/>
-<wire x1="3.6576" y1="24.7904" x2="2.7432" y2="25.7048" width="0.4064" layer="1"/>
-<wire x1="2.7432" y1="27.0256" x2="2.7432" y2="25.7048" width="0.4064" layer="1"/>
+<wire x1="7.8896" y1="22.5136" x2="7.8896" y2="23.8096" width="0.4064" layer="1"/>
+<wire x1="7.8896" y1="23.8096" x2="6.2992" y2="25.4" width="0.4064" layer="1"/>
+<wire x1="5.588" y1="25.4" x2="6.2992" y2="25.4" width="0.4064" layer="1"/>
 </signal>
 <signal name="N$24">
 <contactref element="JP2" pad="1"/>
 <contactref element="K2" pad="5"/>
-<wire x1="5.2832" y1="27.0256" x2="5.2832" y2="26.0096" width="0.4064" layer="1"/>
-<wire x1="5.2832" y1="26.0096" x2="5.6896" y2="25.6032" width="0.4064" layer="1"/>
-<wire x1="5.6896" y1="25.6032" x2="8.9408" y2="25.6032" width="0.4064" layer="1"/>
-<wire x1="8.9408" y1="25.6032" x2="10.0896" y2="24.4544" width="0.4064" layer="1"/>
-<wire x1="10.0896" y1="22.5136" x2="10.0896" y2="24.4544" width="0.4064" layer="1"/>
+<wire x1="10.0896" y1="22.5136" x2="10.0896" y2="23.6416" width="0.4064" layer="1"/>
+<wire x1="10.0896" y1="23.6416" x2="6.9088" y2="26.8224" width="0.4064" layer="1"/>
+<wire x1="6.9088" y1="26.8224" x2="4.4704" y2="26.8224" width="0.4064" layer="1"/>
+<wire x1="4.4704" y1="26.8224" x2="3.048" y2="25.4" width="0.4064" layer="1"/>
 </signal>
 <signal name="N$25">
@@
 <contactref element="JP3" pad="2"/>
 <contactref element="K3" pad="6"/>
-<wire x1="18.8624" y1="22.5136" x2="18.8624" y2="24.4192" width="0.4064" layer="1"/>
-<wire x1="18.8624" y1="24.4192" x2="18.4912" y2="24.7904" width="0.4064" layer="1"/>
-<wire x1="18.4912" y1="24.7904" x2="11.2776" y2="24.7904" width="0.4064" layer="1"/>
-<wire x1="11.2776" y1="24.7904" x2="9.0424" y2="27.0256" width="0.4064" layer="1"/>
+<wire x1="18.8624" y1="22.5136" x2="18.8624" y2="23.6064" width="0.4064" layer="1"/>
+<wire x1="18.8624" y1="23.6064" x2="17.0688" y2="25.4" width="0.4064" layer="1"/>
+<wire x1="17.0688" y1="25.4" x2="13.1064" y2="25.4" width="0.4064" layer="1"/>
 </signal>
 <signal name="N$27">
 <contactref element="JP3" pad="1"/>
 <contactref element="K3" pad="5"/>
-<wire x1="11.5824" y1="27.0256" x2="13.0048" y2="25.6032" width="0.4064" layer="1"/>
-<wire x1="13.0048" y1="25.6032" x2="20.1168" y2="25.6032" width="0.4064" layer="1"/>
-<wire x1="20.1168" y1="25.6032" x2="21.0624" y2="24.6576" width="0.4064" layer="1"/>
-<wire x1="21.0624" y1="22.5136" x2="21.0624" y2="24.6576" width="0.4064" layer="1"/>
+<wire x1="21.0624" y1="22.5136" x2="21.0624" y2="23.6416" width="0.4064" layer="1"/>
+<wire x1="21.0624" y1="23.6416" x2="17.8816" y2="26.8224" width="0.4064" layer="1"/>
+<wire x1="17.8816" y1="26.8224" x2="11.9888" y2="26.8224" width="0.4064" layer="1"/>
+<wire x1="11.9888" y1="26.8224" x2="10.5664" y2="25.4" width="0.4064" layer="1"/>
 </signal>
 <signal name="IO2_EN">

Commit message: hw: rc5
Parts:
- moved LED5 1.63 mm to (11.8, 32.3)
- moved R22 1.63 mm to (11.8, 30.9)
- moved LED4 0.20 mm to (4.27, 32.3)
- moved R21 0.20 mm to (4.27, 30.9)
Routing:
- net LED_IO2: track 51.1 -> 49.5 mm
Changed lines of the file:
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@@
 <layer number="39" name="tKeepout" color="4" fill="11" visible="no" active="yes"/>
 <layer number="40" name="bKeepout" color="1" fill="11" visible="no" active="yes"/>
-<layer number="41" name="tRestrict" color="4" fill="10" visible="no" active="yes"/>
-<layer number="42" name="bRestrict" color="1" fill="10" visible="no" active="yes"/>
+<layer number="41" name="tRestrict" color="4" fill="10" visible="yes" active="yes"/>
+<layer number="42" name="bRestrict" color="1" fill="10" visible="yes" active="yes"/>
 <layer number="43" name="vRestrict" color="2" fill="10" visible="no" active="yes"/>
 <layer number="44" name="Drills" color="7" fill="1" visible="no" active="yes"/>
@@
 <element name="R19" library="rcl" package="R0603" value="330" x="16.256" y="3.2512" rot="MR180"/>
 <element name="R20" library="rcl" package="R0603" value="330" x="62.7888" y="30.8864" rot="MR0"/>
-<element name="R21" library="rcl" package="R0603" value="330" x="4.064" y="30.8864" rot="MR0"/>
-<element name="R22" library="rcl" package="R0603" value="330" x="10.16" y="30.8864" rot="MR0"/>
+<element name="R21" library="rcl" package="R0603" value="330" x="4.2672" y="30.8864" rot="MR0"/>
+<element name="R22" library="rcl" package="R0603" value="330" x="11.7856" y="30.8864" rot="MR0"/>
 <element name="R23" library="rcl" package="R0603" value="330" x="46.5328" y="30.8864" rot="MR0"/>
 <element name="LED2" library="led" package="SML0805" value="" x="16.256" y="1.8288" rot="MR180"/>
 <element name="LED3" library="led" package="SML0805" value="" x="58.3184" y="30.8864"/>
-<element name="LED4" library="led" package="SML0805" value="" x="4.064" y="32.3088" rot="MR0"/>
-<element name="LED5" library="led" package="SML0805" value="" x="10.16" y="32.3088" rot="MR0"/>
+<element name="LED4" library="led" package="SML0805" value="" x="4.2672" y="32.3088" rot="MR0"/>
+<element name="LED5" library="led" package="SML0805" value="" x="11.7856" y="32.3088" rot="MR0"/>
 <element name="LED6" library="led" package="SML0805" value="" x="46.5328" y="32.3088" rot="MR0"/>
 <element name="C16" library="rcl" package="C0805" value=".1u" x="42.4688" y="19.5072" rot="R180"/>
@@
 <contactref element="R21" pad="2"/>
 <contactref element="LED4" pad="A"/>
-<wire x1="3.214" y1="30.8864" x2="3.214" y2="31.5332" width="0.4064" layer="16"/>
-<wire x1="3.214" y1="31.5332" x2="3.014" y2="31.7332" width="0.4064" layer="16"/>
-<wire x1="3.014" y1="32.3088" x2="3.014" y2="31.7332" width="0.4064" layer="16"/>
+<wire x1="3.4172" y1="30.8864" x2="3.4172" y2="31.5332" width="0.4064" layer="16"/>
+<wire x1="3.4172" y1="31.5332" x2="3.2172" y2="31.7332" width="0.4064" layer="16"/>
+<wire x1="3.2172" y1="32.3088" x2="3.2172" y2="31.7332" width="0.4064" layer="16"/>
 </signal>
 <signal name="N$32">
 <contactref element="R22" pad="2"/>
 <contactref element="LED5" pad="A"/>
-<wire x1="9.31" y1="30.8864" x2="9.31" y2="31.5332" width="0.4064" layer="16"/>
-<wire x1="9.31" y1="31.5332" x2="9.11" y2="31.7332" width="0.4064" layer="16"/>
-<wire x1="9.11" y1="32.3088" x2="9.11" y2="31.7332" width="0.4064" layer="16"/>
+<wire x1="10.9356" y1="30.8864" x2="10.9356" y2="31.5332" width="0.4064" layer="16"/>
+<wire x1="10.9356" y1="31.5332" x2="10.7356" y2="31.7332" width="0.4064" layer="16"/>
+<wire x1="10.7356" y1="32.3088" x2="10.7356" y2="31.7332" width="0.4064" layer="16"/>
 </signal>
 <signal name="N$33">
@@
 <signal name="LED_IO1">
 <contactref element="R21" pad="1"/>
-<wire x1="4.914" y1="30.8864" x2="4.8768" y2="30.8864" width="0.2032" layer="16"/>
-<wire x1="4.8768" y1="30.8864" x2="5.8928" y2="29.8704" width="0.2032" layer="16"/>
-<wire x1="5.8928" y1="29.8704" x2="11.3792" y2="29.8704" width="0.2032" layer="16"/>
-<wire x1="11.3792" y1="29.8704" x2="13.0048" y2="28.2448" width="0.2032" layer="16"/>
-<wire x1="13.0048" y1="28.2448" x2="18.4912" y2="28.2448" width="0.2032" layer="16"/>
+<wire x1="5.1172" y1="30.8864" x2="5.08" y2="30.8864" width="0.2032" layer="16"/>
+<wire x1="5.08" y1="30.8864" x2="6.096" y2="29.8704" width="0.2032" layer="16"/>
+<wire x1="6.096" y1="29.8704" x2="13.0048" y2="29.8704" width="0.2032" layer="16"/>
+<wire x1="13.0048" y1="29.8704" x2="14.6304" y2="28.2448" width="0.2032" layer="16"/>
+<wire x1="14.6304" y1="28.2448" x2="18.4912" y2="28.2448" width="0.2032" layer="16"/>
 <wire x1="18.4912" y1="28.2448" x2="19.304" y2="29.0576" width="0.2032" layer="16"/>
 <wire x1="19.304" y1="29.0576" x2="53.848" y2="29.0576" width="0.2032" layer="16"/>
@@
 <contactref element="IC1" pad="26"/>
 <contactref element="R22" pad="1"/>
-<wire x1="11.01" y1="30.8864" x2="10.9728" y2="30.8864" width="0.2032" layer="16"/>
-<wire x1="10.9728" y1="30.8864" x2="13.208" y2="28.6512" width="0.2032" layer="16"/>
-<wire x1="13.208" y1="28.6512" x2="18.288" y2="28.6512" width="0.2032" layer="16"/>
+<wire x1="12.6356" y1="30.8864" x2="12.5984" y2="30.8864" width="0.2032" layer="16"/>
+<wire x1="12.5984" y1="30.8864" x2="14.8336" y2="28.6512" width="0.2032" layer="16"/>
+<wire x1="14.8336" y1="28.6512" x2="18.288" y2="28.6512" width="0.2032" layer="16"/>
 <wire x1="18.288" y1="28.6512" x2="19.1008" y2="29.464" width="0.2032" layer="16"/>
 <wire x1="19.1008" y1="29.464" x2="54.0512" y2="29.464" width="0.2032" layer="16"/>

Commit message: hw: rc6
Routing:
- net LED_IO2: track 49.5 -> 50.8 mm
- net IO2_EN: track 59.3 -> 58.3 mm
- net POWER_EN: track 74.7 -> 73.8 mm
- net LED_POWER: track 75.4 -> 74.5 mm
- net LED_IO1: track 65.5 -> 66.3 mm
Other:
- board text added: "BP"
- board text added: "IO1"
- board text added: "IO2"
- board text added: "PWR"
- board text added: "USB1"
- board text added: "USB2"
- board text added: "_"
- board text added: "rev0"

Commit message: hw: rc7
Parts:
- R24, R26: value 10k -> 56k
- R28: value 10k -> 270k
Changed lines of the file:
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@@
 <element name="C18" library="rcl" package="C0805" value=".1u" x="20.1168" y="7.9248"/>
 <element name="C19" library="rcl" package="C0805" value=".1u" x="8.9408" y="2.6416" rot="MR180"/>
-<element name="R24" library="rcl" package="R0603" value="10k" x="43.688" y="4.2672" rot="MR90"/>
+<element name="R24" library="rcl" package="R0603" value="56k" x="43.688" y="4.2672" rot="MR90"/>
 <element name="R25" library="rcl" package="R0603" value="10k" x="40.8432" y="4.2672" rot="MR270"/>
 <element name="C20" library="rcl" package="C0805" value=".1u" x="39.4208" y="4.2672" rot="MR270"/>
-<element name="R26" library="rcl" package="R0603" value="10k" x="33.1216" y="4.2672" rot="MR90"/>
+<element name="R26" library="rcl" package="R0603" value="56k" x="33.1216" y="4.2672" rot="MR90"/>
 <element name="R27" library="rcl" package="R0603" value="10k" x="35.9664" y="4.2672" rot="MR270"/>
 <element name="C21" library="rcl" package="C0805" value=".1u" x="37.3888" y="4.2672" rot="MR270"/>
-<element name="R28" library="rcl" package="R0603" value="10k" x="24.9936" y="4.2672" rot="MR90"/>
+<element name="R28" library="rcl" package="R0603" value="270k" x="24.9936" y="4.2672" rot="MR90"/>
 <element name="R29" library="rcl" package="R0603" value="10k" x="26.416" y="4.2672" rot="MR270"/>
 <element name="C22" library="rcl" package="C0805" value=".1u" x="27.8384" y="4.2672" rot="MR270"/>

Commit message: hw: rc8
Parts:
- R24, R26: value 56k -> 33k
- R25, R27, R29: value 10k -> 5k6
- R28: value 270k -> 180k
Changed lines of the file:
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@@
 <element name="C18" library="rcl" package="C0805" value=".1u" x="20.1168" y="7.9248"/>
 <element name="C19" library="rcl" package="C0805" value=".1u" x="8.9408" y="2.6416" rot="MR180"/>
-<element name="R24" library="rcl" package="R0603" value="56k" x="43.688" y="4.2672" rot="MR90"/>
-<element name="R25" library="rcl" package="R0603" value="10k" x="40.8432" y="4.2672" rot="MR270"/>
+<element name="R24" library="rcl" package="R0603" value="33k" x="43.688" y="4.2672" rot="MR90"/>
+<element name="R25" library="rcl" package="R0603" value="5k6" x="40.8432" y="4.2672" rot="MR270"/>
 <element name="C20" library="rcl" package="C0805" value=".1u" x="39.4208" y="4.2672" rot="MR270"/>
-<element name="R26" library="rcl" package="R0603" value="56k" x="33.1216" y="4.2672" rot="MR90"/>
-<element name="R27" library="rcl" package="R0603" value="10k" x="35.9664" y="4.2672" rot="MR270"/>
+<element name="R26" library="rcl" package="R0603" value="33k" x="33.1216" y="4.2672" rot="MR90"/>
+<element name="R27" library="rcl" package="R0603" value="5k6" x="35.9664" y="4.2672" rot="MR270"/>
 <element name="C21" library="rcl" package="C0805" value=".1u" x="37.3888" y="4.2672" rot="MR270"/>
-<element name="R28" library="rcl" package="R0603" value="270k" x="24.9936" y="4.2672" rot="MR90"/>
-<element name="R29" library="rcl" package="R0603" value="10k" x="26.416" y="4.2672" rot="MR270"/>
+<element name="R28" library="rcl" package="R0603" value="180k" x="24.9936" y="4.2672" rot="MR90"/>
+<element name="R29" library="rcl" package="R0603" value="5k6" x="26.416" y="4.2672" rot="MR270"/>
 <element name="C22" library="rcl" package="C0805" value=".1u" x="27.8384" y="4.2672" rot="MR270"/>
 <element name="R30" library="rcl" package="R0603" value="330" x="62.7888" y="32.3088" rot="MR0"/>

Commit message: hw: update hammond library
Parts:
- BOX2: device hammond:1151K -> hammond:1551K
Changed lines of the file:
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@@
 <element name="X3" library="con-phoenix-381_l" package="MC2" value="MC2" x="20.9296" y="4.8768"/>
 <element name="U1" library="SparkFun-PowerIC" package="SOT23-5" value="MIC5301" x="56.6928" y="8.9408"/>
-<element name="BOX2" library="hammond" package="1151K" value="HAMMOND-BOX-K" x="0" y="0" locked="yes"/>
+<element name="BOX2" library="hammond" package="1551K" value="HAMMOND-BOX-K" x="0" y="0" locked="yes"/>
 <element name="D2" library="diode" package="SOT23" value="BAT54" x="3.048" y="10.9728" rot="MR180"/>
 <element name="Q1" library="SparkFun-DiscreteSemi" package="SOT23-3" value="BSS138" x="6.2992" y="10.9728" rot="MR0">
