File: hardware/power-manager.brd (EAGLE design)
At the start: 74 x 34 mm, 90 parts, among them IC1 ATMEGA168-AU, K1 G6J-2FL-Y, K2 G6J-2FL-Y, K3 G6J-2FL-Y, Q1 BSS138, Q2 BSS138, Q3 BSS138, U1 MIC5301, U2 INA219, U3 TPS2552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

Commit message: hw: update part values
Parts:
- R12, R8: value 10k -> 22k
- R4, R5, R6: value 10k -> 5k6
Changed lines of the file:
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@@
 <?xml version="1.0" encoding="utf-8"?>
 <!DOCTYPE eagle SYSTEM "eagle.dtd">
-<eagle version="6.3">
+<eagle version="6.4">
 <drawing>
 <settings>
@@
 <element name="C8" library="rcl" package="C0805" value="22p" x="70.7136" y="14.4272" rot="MR180"/>
 <element name="ISP1" library="balto" package="2X03" value="" x="70.7136" y="21.7424" rot="R270"/>
-<element name="R4" library="rcl" package="R0603" value="10k" x="70.7136" y="17.0688" rot="R180"/>
-<element name="R5" library="rcl" package="R0603" value="10k" x="25.4" y="12.192" rot="R225"/>
-<element name="R6" library="rcl" package="R0603" value="10k" x="24.384" y="13.208" rot="R225"/>
+<element name="R4" library="rcl" package="R0603" value="5k6" x="70.7136" y="17.0688" rot="R180"/>
+<element name="R5" library="rcl" package="R0603" value="5k6" x="25.4" y="12.192" rot="R225"/>
+<element name="R6" library="rcl" package="R0603" value="5k6" x="24.384" y="13.208" rot="R225"/>
 <element name="U$2" library="SparkFun-Connectors" package="USB-MINIB" value="USB-MINIB-5PIN" x="44.5008" y="4.4704" rot="R90"/>
 <element name="R7" library="rcl" package="R0603" value="330" x="29.8704" y="30.8864" rot="MR0"/>
 <element name="C9" library="rcl" package="C0805" value=".1u" x="40.8432" y="9.3472" rot="R180"/>
-<element name="R8" library="rcl" package="R0603" value="10k" x="52.0192" y="15.4432" rot="R90"/>
+<element name="R8" library="rcl" package="R0603" value="22k" x="52.0192" y="15.4432" rot="R90"/>
 <element name="C10" library="rcl" package="C0805" value=".1u" x="45.9232" y="17.0688" rot="R90"/>
 <element name="R9" library="rcl" package="R0603" value="10" x="48.1584" y="16.256"/>
@@
 <element name="U$3" library="SparkFun-Connectors" package="USB-MINIB" value="USB-MINIB-5PIN" x="32.3088" y="4.4704" rot="R90"/>
 <element name="C11" library="rcl" package="C0805" value=".1u" x="28.6512" y="9.3472" rot="R180"/>
-<element name="R12" library="rcl" package="R0603" value="10k" x="35.3568" y="15.4432" rot="R90"/>
+<element name="R12" library="rcl" package="R0603" value="22k" x="35.3568" y="15.4432" rot="R90"/>
 <element name="C12" library="rcl" package="C0805" value=".1u" x="29.2608" y="17.0688" rot="R90"/>
 <element name="R13" library="rcl" package="R0603" value="10" x="31.496" y="16.256"/>
@@
 </signal>
 </signals>
-<errors>
-</errors>
 </board>
 </drawing>

Commit message: hw: add notes and pdf
Parts:
- K1, K2, K3: value G6J-2FL-Y -> IM03GR
Changed lines of the file:
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@@
 <element name="JP1" library="SparkFun-Connectors" package="1X02" value="" x="52.4256" y="2.2352" rot="R90"/>
 <element name="U2" library="balto" package="SOT23-8L" value="INA219" x="42.4688" y="17.0688" rot="R90"/>
-<element name="K1" library="relay" package="G6J-2FL-Y" value="G6J-2FL-Y" x="5.6896" y="10.9728">
+<element name="K1" library="relay" package="G6J-2FL-Y" value="IM03GR" x="5.6896" y="10.9728">
 <attribute name="OC_NEWARK" value="04M9907" x="99.6696" y="-135.0772" size="1.778" layer="27" display="off"/>
 <attribute name="MPN" value="G6J-2FL-Y-TR DC4.5" x="99.6696" y="-135.0772" size="1.778" layer="27" display="off"/>
@@
 <element name="C15" library="rcl" package="C0805" value=".1u" x="34.7472" y="19.5072"/>
 <element name="D1" library="diode" package="SOT23" value="BAT54" x="3.048" y="19.9136" rot="MR180"/>
-<element name="K2" library="relay" package="G6J-2FL-Y" value="G6J-2FL-Y" x="5.6896" y="19.9136">
+<element name="K2" library="relay" package="G6J-2FL-Y" value="IM03GR" x="5.6896" y="19.9136">
 <attribute name="OC_NEWARK" value="04M9907" x="111.0996" y="-126.1364" size="1.778" layer="27" display="off"/>
 <attribute name="MPN" value="G6J-2FL-Y-TR DC4.5" x="111.0996" y="-126.1364" size="1.778" layer="27" display="off"/>
@@
 <element name="JP2" library="SparkFun-Connectors" package="1X02" value="" x="3.048" y="25.4"/>
 <element name="D3" library="diode" package="SOT23" value="BAT54" x="14.0208" y="19.9136" rot="MR180"/>
-<element name="K3" library="relay" package="G6J-2FL-Y" value="G6J-2FL-Y" x="16.6624" y="19.9136">
+<element name="K3" library="relay" package="G6J-2FL-Y" value="IM03GR" x="16.6624" y="19.9136">
 <attribute name="OC_NEWARK" value="04M9907" x="133.5024" y="-126.1364" size="1.778" layer="27" display="off"/>
 <attribute name="MPN" value="G6J-2FL-Y-TR DC4.5" x="133.5024" y="-126.1364" size="1.778" layer="27" display="off"/>

Commit message: hw: update xtal cap values to 33p
Parts:
- C7, C8: value 22p -> 33p
Changed lines of the file:
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@@
 <element name="C6" library="rcl" package="C0805" value=".1u" x="62.992" y="30.8864" rot="R90"/>
 <element name="Y1" library="SparkFun-FreqCtrl" package="CRYSTAL-SMD-5X3" value="12MHz" x="70.7136" y="12.3952" rot="R90"/>
-<element name="C7" library="rcl" package="C0805" value="22p" x="70.7136" y="10.3632" rot="MR0"/>
-<element name="C8" library="rcl" package="C0805" value="22p" x="70.7136" y="14.4272" rot="MR180"/>
+<element name="C7" library="rcl" package="C0805" value="33p" x="70.7136" y="10.3632" rot="MR0"/>
+<element name="C8" library="rcl" package="C0805" value="33p" x="70.7136" y="14.4272" rot="MR180"/>
 <element name="ISP1" library="balto" package="2X03" value="" x="70.7136" y="21.7424" rot="R270"/>
 <element name="R4" library="rcl" package="R0603" value="5k6" x="70.7136" y="17.0688" rot="R180"/>
